Commit message: Changing z offset for flange
Aiming to remove the issue with z offset, likely due to where we are defining flange

File: BAE_system_description/urdf/bae_system.urdf.xacro (robot description, xacro)
@@ -24,5 +24,5 @@
     <parent link="lbr_link_ee"/>
     <child link="zivid_base_link" />
-    <origin xyz="0 0 0" rpy="0 0 -1.5708" />
+    <origin xyz="0 0 0.006" rpy="0 0 -1.5708" />
   </joint>
   <joint name="zivid_camera_joint" type="fixed">
